File: rp2350a_main_board.kicad_pcb (KiCad board)
At the start: 2 copper layers, 63.5 x 40.6 mm, 75 parts, among them J1 USB_C_Receptacle_USB2.0_16P, J2 SM03B-SRSS-TB, J3 Micro_SD_Card_Det1, J4 SM03B-SRSS-TB, J5 Conn_02x12, J6 Conn_02x12, J7 Conn_02x12, J8 Conn_02x12, SW1 SW_SPDT, SW2 SW_Push, SW3 SW_Push, U1 TPS63802, U2 TPS2116DRL, U3 W25Q16JVSS, U4 RP2350_60QFN, U5 APS1604M-3SQRx-SN, Y1 ABM8-272-T3

Commit message: Update PCB components, board version, and numbering
Parts:
- added C23: 10u, Capacitor_SMD:C_0603_1608Metric_Pad1.08x0.95mm_HandSolder, F.Cu at (78.7, 33.0)
- added C24: 10u, Capacitor_SMD:C_0603_1608Metric_Pad1.08x0.95mm_HandSolder, F.Cu at (102.6, 39.8)
- added C25: 10u, Capacitor_SMD:C_0603_1608Metric_Pad1.08x0.95mm_HandSolder, F.Cu at (102.6, 38.4)
- added C26: 1u, Capacitor_SMD:C_0402_1005Metric_Pad0.74x0.62mm_HandSolder, F.Cu at (98.9, 48.1)
- added J10: Conn_02x12, Connector_PinSocket_2.54mm:PinSocket_2x12_P2.54mm_Vertical_SMD, B.Cu at (85.1, 45.7)
- added J9: Conn_02x12, Connector_PinSocket_2.54mm:PinSocket_2x12_P2.54mm_Vertical_SMD, B.Cu at (29.2, 45.7)
- added TP4: PR, TestPoint:TestPoint_Pad_D1.0mm, F.Cu at (93.6, 39.6)
- added TP5: MODE, TestPoint:TestPoint_Pad_D1.0mm, F.Cu at (93.6, 42.7)
- added U6: USBLC6-2SC6, Package_TO_SOT_SMD:SOT-23-6, F.Cu at (65.0, 37.5)
- L1: value 470n -> XFL4015-471MEC
- R14: value 33k -> 0
- R17: value 10k -> 0
- U2: value TPS2116DRL -> TPS2117DRL
- moved TP3 29.0 mm to (106.4, 38.2)
- moved TP2 28.4 mm to (96.1, 50.3)
- moved TP1 26.4 mm to (96.4, 47.8)
- moved R14 25.6 mm to (100.1, 41.5), turned to -90 degrees
- moved R17 22.0 mm to (96.3, 40.2), turned to 90 degrees
- moved U2 21.2 mm to (98.2, 40.2)
- moved R16 21.0 mm to (100.1, 38.9)
Connections:
- R14 pad 1: VUSB -> Net-(U2-MODE)
- R14 pad 2: Net-(U2-PR1) -> GND
- U2 pad 5: VUSB -> Net-(U2-MODE)
Routing:
- net VIN: track 26.1 -> 13.0 mm
- net Net-(U2-ST): track 7.17 -> 0.00 mm, vias 2 -> 1
- net VUSB: track 38.9 -> 31.9 mm
- net Net-(U1-EN): track 7.77 -> 1.87 mm, vias 0 -> 1
- net Net-(SW1-A): track 5.06 -> 0.00 mm
- net Net-(U1-PG): track 5.38 -> 0.81 mm
- net Net-(U2-PR1): track 4.08 -> 0.00 mm
- net VBAT: track 6.78 -> 2.89 mm
- net /USB_D+: track 15.5 -> 13.2 mm
- net /USB_D-: track 14.2 -> 12.8 mm
- net GND: vias 68 -> 63
Other:
- board text added: "No."
- board text added: "V1.1.0"
- board text removed: "V1.0.0"

Commit message: v1.1.0 WIP
Parts:
- R15: footprint Resistor_SMD:R_0603_1608Metric_Pad0.98x0.95mm_HandSolder -> Resistor_SMD:R_0402_1005Metric_Pad0.72x0.64mm_HandSolder
- TP1, TP2, TP3, TP4, TP5: moved to B.Cu
- moved TP3 31.1 mm to (75.8, 32.6), turned to 180 degrees
- moved C24 28.9 mm to (74.0, 35.6), turned to 90 degrees
- moved R16 26.1 mm to (74.7, 33.3), turned to 180 degrees
- moved TP2 24.7 mm to (73.8, 39.9), turned to 180 degrees
- moved C25 24.4 mm to (78.4, 35.6), turned to 90 degrees
- moved C26 23.7 mm to (76.5, 40.6), turned to 180 degrees
- moved R14 23.0 mm to (77.5, 37.7), turned to 180 degrees
- moved U2 22.5 mm to (76.2, 35.6)
- moved R17 21.5 mm to (74.9, 37.7), turned to 0 degrees
- moved TP1 21.3 mm to (76.6, 39.9), turned to 180 degrees
- moved TP4 19.4 mm to (74.3, 37.7), turned to 180 degrees
- moved TP5 16.3 mm to (78.1, 37.7), turned to 180 degrees
- moved C3 4.89 mm to (71.9, 47.4)
- moved C1 4.06 mm to (78.0, 45.2), turned to -90 degrees
- moved R1 3.57 mm to (77.3, 42.3), turned to 90 degrees
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Connections:
- J10 pad 14: unconnected-(J10-Pin_14-Pad14) -> GND
- J10 pad 2: unconnected-(J10-Pin_2-Pad2) -> VUSB
- J10 pad 20: unconnected-(J10-Pin_20-Pad20) -> GND
- J10 pad 24: unconnected-(J10-Pin_24-Pad24) -> GND
- J10 pad 3: unconnected-(J10-Pin_3-Pad3) -> VBAT
- J10 pad 6: unconnected-(J10-Pin_6-Pad6) -> VIN
- J10 pad 7: unconnected-(J10-Pin_7-Pad7) -> +3V3
- J9 pad 1: unconnected-(J9-Pin_1-Pad1) -> +3V3
- J9 pad 11: unconnected-(J9-Pin_11-Pad11) -> GND
- J9 pad 17: unconnected-(J9-Pin_17-Pad17) -> GND
- J9 pad 23: unconnected-(J9-Pin_23-Pad23) -> GND
- J9 pad 3: unconnected-(J9-Pin_3-Pad3) -> +3V3
- J9 pad 5: unconnected-(J9-Pin_5-Pad5) -> GND
Routing:
- net VUSB: track 31.9 -> 58.0 mm, vias 3 -> 4
- net VIN: track 13.0 -> 32.7 mm, vias 1 -> 0
- net Net-(SW1-A): track 0.00 -> 9.06 mm
- net VBAT: track 2.89 -> 10.3 mm
- net Net-(U2-ST): track 0.00 -> 4.68 mm, vias 1 -> 2
- net Net-(D1-A): track 3.85 -> 8.50 mm
- net +3V3: track 186.9 -> 191.5 mm, vias 13 -> 12
- net /QSPI_SS: track 41.3 -> 45.4 mm
- net Net-(U1-EN): track 1.87 -> 5.84 mm
- net /RUN: track 73.7 -> 70.1 mm
- net /GPIO15: track 48.7 -> 45.7 mm
- net /USB_D+: track 13.2 -> 15.5 mm
- net /USB_D-: track 12.8 -> 15.0 mm
- net Net-(U2-PR1): track 0.00 -> 1.95 mm, vias 0 -> 1
- net Net-(U2-MODE): track 0.00 -> 1.89 mm, vias 0 -> 1
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Other:
- board text added: "9"
- board text added: "MODE"
- board text added: "PR1"
- board text added: "비 오는 날 유독 심하다"
- board text removed: "9 RUN"

Commit message: Update BOM
Changed lines of the file:
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@@
 		(sheetname "/")
 		(sheetfile "rp2350a_main_board.kicad_sch")
-		(attr smd exclude_from_bom)
+		(attr smd)
 		(fp_line
 			(start 4.7 2)
@@
 	(gr_poly
 		(pts
-			(xy 73.279 56.388) (xy 73.406 56.515) (xy 74.168 56.515) (xy 74.295 56.388) (xy 74.168 56.261) (xy 73.406 56.261)
+			(xy 72.644 56.515) (xy 72.771 56.642) (xy 73.533 56.642) (xy 73.66 56.515) (xy 73.533 56.388) (xy 72.771 56.388)
 		)
 		(stroke
@@
 	(gr_poly
 		(pts
-			(xy 73.152 56.515) (xy 73.025 56.642) (xy 73.025 57.404) (xy 73.152 57.531) (xy 73.279 57.404) (xy 73.279 56.642)
+			(xy 72.517 56.642) (xy 72.39 56.769) (xy 72.39 57.531) (xy 72.517 57.658) (xy 72.644 57.531) (xy 72.644 56.769)
 		)
 		(stroke
@@
 		(layer "F.SilkS")
 	)
+	(gr_rect
+		(start 26.61 45.72)
+		(end 37.465 50.8)
+		(stroke
+			(width 0.1)
+			(type default)
+		)
+		(fill no)
+		(layer "F.SilkS")
+	)
 	(gr_line
 		(start 48.387 63.627)
@@
 	(gr_poly
 		(pts
-			(xy 74.422 56.515) (xy 74.295 56.642) (xy 74.295 57.404) (xy 74.422 57.531) (xy 74.549 57.404) (xy 74.549 56.642)
+			(xy 73.787 56.642) (xy 73.66 56.769) (xy 73.66 57.531) (xy 73.787 57.658) (xy 73.914 57.531) (xy 73.914 56.769)
 		)
 		(stroke
@@
 	(gr_poly
 		(pts
-			(xy 74.422 55.245) (xy 74.295 55.372) (xy 74.295 56.134) (xy 74.422 56.261) (xy 74.549 56.134) (xy 74.549 55.372)
+			(xy 73.787 55.372) (xy 73.66 55.499) (xy 73.66 56.261) (xy 73.787 56.388) (xy 73.914 56.261) (xy 73.914 55.499)
 		)
 		(stroke
@@
 	(gr_poly
 		(pts
-			(xy 73.279 57.658) (xy 73.406 57.785) (xy 74.168 57.785) (xy 74.295 57.658) (xy 74.168 57.531) (xy 73.406 57.531)
+			(xy 72.644 57.785) (xy 72.771 57.912) (xy 73.533 57.912) (xy 73.66 57.785) (xy 73.533 57.658) (xy 72.771 57.658)
 		)
 		(stroke
@@
 	(gr_poly
 		(pts
-			(xy 75.184 55.118) (xy 75.311 55.245) (xy 76.073 55.245) (xy 76.2 55.118) (xy 76.073 54.991) (xy 75.311 54.991)
+			(xy 74.549 55.245) (xy 74.676 55.372) (xy 75.438 55.372) (xy 75.565 55.245) (xy 75.438 55.118) (xy 74.676 55.118)
 		)
 		(stroke
@@
 	(gr_poly
 		(pts
-			(xy 76.327 56.515) (xy 76.2 56.642) (xy 76.2 57.404) (xy 76.327 57.531) (xy 76.454 57.404) (xy 76.454 56.642)
+			(xy 75.692 56.642) (xy 75.565 56.769) (xy 75.565 57.531) (xy 75.692 57.658) (xy 75.819 57.531) (xy 75.819 56.769)
 		)
 		(stroke
@@
 	(gr_poly
 		(pts
-			(xy 76.327 55.245) (xy 76.2 55.372) (xy 76.2 56.134) (xy 76.327 56.261) (xy 76.454 56.134) (xy 76.454 55.372)
+			(xy 75.692 55.372) (xy 75.565 55.499) (xy 75.565 56.261) (xy 75.692 56.388) (xy 75.819 56.261) (xy 75.819 55.499)
 		)
 		(stroke
@@
 		(layer "F.SilkS")
 	)
+	(gr_rect
+		(start 26.61 53.34)
+		(end 37.465 58.42)
+		(stroke
+			(width 0.1)
+			(type default)
+		)
+		(fill no)
+		(layer "F.SilkS")
+	)
 	(gr_poly
 		(pts
-			(xy 75.184 57.658) (xy 75.311 57.785) (xy 76.073 57.785) (xy 76.2 57.658) (xy 76.073 57.531) (xy 75.311 57.531)
+			(xy 74.549 57.785) (xy 74.676 57.912) (xy 75.438 57.912) (xy 75.565 57.785) (xy 75.438 57.658) (xy 74.676 57.658)
 		)
 		(stroke
@@
 	(gr_poly
 		(pts
-			(xy 73.279 55.118) (xy 73.406 55.245) (xy 74.168 55.245) (xy 74.295 55.118) (xy 74.168 54.991) (xy 73.406 54.991)
+			(xy 72.644 55.245) (xy 72.771 55.372) (xy 73.533 55.372) (xy 73.66 55.245) (xy 73.533 55.118) (xy 72.771 55.118)
 		)
 		(stroke
@@
 	(gr_poly
 		(pts
-			(xy 75.184 56.388) (xy 75.311 56.515) (xy 76.073 56.515) (xy 76.2 56.388) (xy 76.073 56.261) (xy 75.311 56.261)
+			(xy 74.549 56.515) (xy 74.676 56.642) (xy 75.438 56.642) (xy 75.565 56.515) (xy 75.438 56.388) (xy 74.676 56.388)
 		)
 		(stroke
@@
 	(gr_poly
 		(pts
-			(xy 75.057 55.245) (xy 74.93 55.372) (xy 74.93 56.134) (xy 75.057 56.261) (xy 75.184 56.134) (xy 75.184 55.372)
+			(xy 74.422 55.372) (xy 74.295 55.499) (xy 74.295 56.261) (xy 74.422 56.388) (xy 74.549 56.261) (xy 74.549 55.499)
 		)
 		(stroke
@@
 	(gr_poly
 		(pts
-			(xy 73.152 55.245) (xy 73.025 55.372) (xy 73.025 56.134) (xy 73.152 56.261) (xy 73.279 56.134) (xy 73.279 55.372)
+			(xy 72.517 55.372) (xy 72.39 55.499) (xy 72.39 56.261) (xy 72.517 56.388) (xy 72.644 56.261) (xy 72.644 55.499)
 		)
 		(stroke
@@
 	(gr_poly
 		(pts
-			(xy 75.057 56.515) (xy 74.93 56.642) (xy 74.93 57.404) (xy 75.057 57.531) (xy 75.184 57.404) (xy 75.184 56.642)
+			(xy 74.422 56.642) (xy 74.295 56.769) (xy 74.295 57.531) (xy 74.422 57.658) (xy 74.549 57.531) (xy 74.549 56.769)
 		)
 		(stroke
@@
 		)
 	)
+	(gr_text "FLASH"
+		(at 50.038 41.529 90)
+		(layer "F.SilkS")
+		(effects
+			(font
+				(size 0.6096 0.6096)
+				(thickness 0.1524)
+				(bold yes)
+			)
+			(justify left bottom)
+		)
+	)
 	(gr_text "Main Board"
 		(at 57.15 63.881 0)
@@
 		)
 	)
+	(gr_text "PSRAM"
+		(at 50.8 35.179 90)
+		(layer "F.SilkS")
+		(effects
+			(font
+				(size 0.6096 0.6096)
+				(thickness 0.1524)
+				(bold yes)
+			)
+			(justify left bottom)
+		)
+	)
+	(gr_text "HSTX"
+		(at 39.878 46.355 0)
+		(layer "F.SilkS")
+		(effects
+			(font
+				(size 0.6096 0.6096)
+				(thickness 0.1524)
+				(bold yes)
+			)
+			(justify right)
+		)
+	)
 	(gr_text "12 13"
 		(at 33.655 46.99 0)
@@
 		)
 	)
+	(gr_text "HSTX"
+		(at 39.878 53.975 0)
+		(layer "F.SilkS")
+		(effects
+			(font
+				(size 0.6096 0.6096)
+				(thickness 0.1524)
+				(bold yes)
+			)
+			(justify right)
+		)
+	)
+	(gr_text "GND"
+		(at 32.004 35.687 0)
+		(layer "F.SilkS")
+		(effects
+			(font
+				(size 0.6096 0.6096)
+				(thickness 0.1524)
+				(bold yes)
+			)
+			(justify left)
+		)
+	)
 	(gr_text "No."
-		(at 72.136 57.531 0)
+		(at 72.39 57.658 0)
 		(layer "F.SilkS")
 		(effects
@@
 				(thickness 0.1524)
 			)
+			(justify right)
 		)
 	)
@@
 		)
 	)
+	(gr_text "3V3"
+		(at 33.909 30.48 0)
+		(layer "F.SilkS")
+		(effects
+			(font
+				(size 0.6096 0.6096)
+				(thickness 0.1524)
+				(bold yes)
+			)
+			(justify right)
+		)
+	)
 	(gr_text "C G D"
 		(at 79.121 59.817 0)
@@
 		)
 	)
+	(gr_text "3V3"
+		(at 33.909 33.147 0)
+		(layer "F.SilkS")
+		(effects
+			(font
+				(size 0.6096 0.6096)
+				(thickness 0.1524)
+				(bold yes)
+			)
+			(justify right)
+		)
+	)
 	(gr_text "LOG"
 		(at 68.199 60.96 0)
@@
 	)
 	(segment
+		(start 70.612 40.767)
+		(end 71.755 39.624)
+		(width 0.508)
+		(layer "F.Cu")
+		(net 1)
+	)
+	(segment
 		(start 38.227 38.862)
 		(end 40.259 38.862)
@@
 	)
 	(segment
+		(start 71.755 39.624)
+		(end 71.755 26.67)
+		(width 0.508)
+		(layer "F.Cu")
+		(net 1)
+	)
+	(segment
 		(start 61.195 47.35)
 		(end 61.195 46.882)
@@
 	)
 	(segment
-		(start 71.755 33.401)
-		(end 71.755 26.67)
-		(width 0.508)
-		(layer "F.Cu")
-		(net 1)
-	)
-	(segment
 		(start 60.0035 38.227)
 		(end 60.071 38.1595)
@@
 	)
 	(segment
-		(start 71.755 33.655)
-		(end 71.755 33.401)
-		(width 0.508)
+		(start 57.15 31.685)
+		(end 57.085 31.75)
+		(width 0.254)
 		(layer "F.Cu")
 		(net 1)
 	)
 	(segment
-		(start 57.15 31.685)
-		(end 57.085 31.75)
-		(width 0.254)
+		(start 70.612 44.45)
+		(end 70.612 40.767)
+		(width 0.508)
 		(layer "F.Cu")
 		(net 1)
@@
 	)
 	(segment
-		(start 71.755 39.624)
-		(end 71.755 33.401)
-		(width 0.508)
-		(layer "F.Cu")
-		(net 1)
-	)
-	(segment
 		(start 58.059999 31.75)
 		(end 57.085 31.75)
@@
 	)
 	(segment
-		(start 70.612 44.45)
-		(end 70.612 40.767)
-		(width 0.508)
-		(layer "F.Cu")
-		(net 1)
-	)
-	(segment
 		(start 41.927 40.53)
 		(end 41.927 42.015)
@@
 		(layer "F.Cu")
 		(net 1)
-	)
-	(segment
-		(start 70.612 40.767)
-		(end 71.755 39.624)
-		(width 0.508)
-		(layer "F.Cu")
-		(net 1)
